File: Hardware/Design Files/LautIO.brd (EAGLE design)
At the start: 200 x 150 mm, 223 parts, among them IC1 REG1117, J1 614004134726, J2 614004134726, J3 455-1750-1-ND, J4 455-1750-1-ND, J5 SJ1-3523N, Q1 ZX5T953, Q2 12.288MHz, U1 ADAU1701JSTZ, U2 TDA7498ETR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

Commit message: Final Proto V1 hardware filse
Parts:
- added J7: (no value), SparkFun-Connectors:1X02
Connections:
- net +12V: now also J7.2
- net GND: now also J7.1
Routing:
- net +12V: track 14.3 -> 94.0 mm, vias 12 -> 13
- net GND: vias 425 -> 788
Other:
- board text added: "+12V"
