File: Hardware/Design Files/LautIO.sch (EAGLE design)
At the start: 223 parts, among them IC1 REG1117, J1 614004134726, J2 614004134726, J3 455-1750-1-ND, J4 455-1750-1-ND, J5 SJ1-3523N, Q1 ZX5T953, Q2 12.288MHz, U1 ADAU1701JSTZ, U2 TDA7498ETR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

Commit message: Final Proto V1 hardware filse
Parts:
- added J7: (no value), SparkFun-Connectors:CONN_02
Connections:
- net +12V: now also J7.2
- net GND: now also J7.1
Other:
- note added: "Fan Connector"
Changed lines of the file:
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@@
 <part name="PAD12" library="wirepad" library_urn="urn:adsk.eagle:library:412" deviceset="SMD2" device="" package3d_urn="urn:adsk.eagle:package:30839/1"/>
 <part name="GND49" library="supply1" library_urn="urn:adsk.eagle:library:371" deviceset="GND" device=""/>
+<part name="J7" library="SparkFun-Connectors" deviceset="CONN_02" device=""/>
 </parts>
 <sheets>
@@
 <text x="119.38" y="144.78" size="1.778" layer="97">12V Terminal</text>
 <text x="17.78" y="20.32" size="1.778" layer="97" rot="R270">DSP Potis</text>
+<text x="162.56" y="144.78" size="1.778" layer="97">Fan Connector</text>
 </plain>
 <instances>
@@
 <attribute name="NAME" x="250.317" y="67.8942" size="1.778" layer="95"/>
 <attribute name="VALUE" x="247.523" y="71.882" size="1.778" layer="96" rot="R180"/>
+</instance>
+<instance part="J7" gate="G$1" x="165.1" y="172.72" smashed="yes" rot="R270">
+<attribute name="VALUE" x="160.274" y="175.26" size="1.778" layer="96" font="vector" rot="R270"/>
+<attribute name="NAME" x="170.688" y="175.26" size="1.778" layer="95" font="vector" rot="R270"/>
 </instance>
 </instances>
@@
 <segment>
 <pinref part="X1" gate="-2" pin="KL"/>
-<wire x1="121.92" y1="167.64" x2="121.92" y2="149.86" width="0.1524" layer="91"/>
+<wire x1="121.92" y1="167.64" x2="121.92" y2="162.56" width="0.1524" layer="91"/>
 <pinref part="GND8" gate="1" pin="GND"/>
+<wire x1="121.92" y1="162.56" x2="121.92" y2="149.86" width="0.1524" layer="91"/>
+<wire x1="165.1" y1="165.1" x2="165.1" y2="162.56" width="0.1524" layer="91"/>
+<wire x1="165.1" y1="162.56" x2="121.92" y2="162.56" width="0.1524" layer="91"/>
+<junction x="121.92" y="162.56"/>
+<pinref part="J7" gate="G$1" pin="1"/>
 </segment>
 <segment>
@@
 <segment>
 <pinref part="X1" gate="-1" pin="KL"/>
-<wire x1="114.3" y1="167.64" x2="114.3" y2="149.86" width="0.1524" layer="91"/>
+<wire x1="114.3" y1="167.64" x2="114.3" y2="160.02" width="0.1524" layer="91"/>
 <pinref part="P+5" gate="1" pin="+12V"/>
-</segment>
-</net>
+<wire x1="114.3" y1="160.02" x2="114.3" y2="149.86" width="0.1524" layer="91"/>
+<wire x1="167.64" y1="165.1" x2="167.64" y2="160.02" width="0.1524" layer="91"/>
+<wire x1="167.64" y1="160.02" x2="114.3" y2="160.02" width="0.1524" layer="91"/>
+<junction x="114.3" y="160.02"/>
+<pinref part="J7" gate="G$1" pin="2"/>
+</segment>
+</net>
